File: pcb-design/scale module/V0_3_untested/_V0_3-Scale_Module.kicad_pcb (KiCad board)
At the start: 2 copper layers, 80 x 100 mm, 28 parts, among them J1 ESP32-left-RXTX, J10 PowerIn, J11 Loadcell1-Input, J12 Loadcell2-Input, J13 DS18B20-1, J14 DS18B20-2, J15 SHT40 Ambient, J16 Sound Module INMP441 - Hive2, J17 I2C, J18 Expansion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

Commit message: re-upladed files
Routing:
- net GND: vias 89 -> 88
Other:
- board text added: "L/R"
- board text removed: "L"
- board text removed: "R=3.3V"
Changed lines of the file:
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@@
+		)
+	)
+	(gr_text "L/R"
+		(at 171 48 0)
+		(layer "F.SilkS")
+		(effects
+			(font
+				(size 1 1)
+				(thickness 0.1)
+			)
+			(justify left bottom)
 		)
 	)
@@
 		)
 	)
-	(gr_text "R=3.3V"
-		(at 171.5 68 0)
-		(layer "F.SilkS")
-		(effects
-			(font
-				(size 1 1)
-				(thickness 0.1)
-			)
-			(justify left bottom)
-		)
-	)
-	(gr_text "L"
-		(at 172 48 0)
-		(layer "F.SilkS")
-		(effects
-			(font
-				(size 1 1)
-				(thickness 0.1)
-			)
-			(justify left bottom)
-		)
-	)
 	(gr_text "3.3V"
 		(at 172 65.5 0)
@@
 		)
 	)
+	(gr_text "L/R"
+		(at 172 68 0)
+		(layer "F.SilkS")
+		(effects
+			(font
+				(size 1 1)
+				(thickness 0.1)
+			)
+			(justify left bottom)
+		)
+	)
 	(gr_text "GND"
-		(at 172.5 70.5 0)
+		(at 172 70.5 0)
 		(layer "F.SilkS")
 		(effects
@@
 	)
 	(gr_text "BCLK\nWS\nSD"
-		(at 172.5 78 0)
+		(at 172 78 0)
 		(layer "F.SilkS")
 		(effects
@@
 		(size 0.6)
 		(drill 0.3)
-		(layers "F.Cu" "B.Cu")
-		(free yes)
-		(net "GND")
-	)
-	(via
-		(at 172 71)
-		(size 0.6)
-		(drill 0.3)
