File: pcb-design/power module/_V0_3-Power_Module.kicad_pcb (KiCad board)
At the start: 2 copper layers, 76 x 56 mm, 17 parts, among them J16 SolarPowerIn and INA219, J17 CN3971, J18 TPS63020-GND-OUT, J19 TPS63020-V-IN, J20 ConnectorHiveScale, J21 MAXS17048, J23 TPS63020-3.3V-OUT, J6 TPS63020-GND-IN, m3-bl MountingHole_3.2mm_M3, m3-br MountingHole_3.2mm_M3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

Commit message: added connector for solar panel to power module
Parts:
- added INA219-Solar+1: Solar_Panel_In, TerminalBlock:TerminalBlock_Xinya_XY308-2.54-2P_1x02_P2.54mm_Horizontal, F.Cu at (174.1, 46.4)
- moved stabilizer_usb_1 3.38 mm to (178.8, 44.0)
- moved TP4056+1 3.38 mm to (191.5, 66.9)
- moved TP4056-1 3.38 mm to (181.3, 66.9)
- moved stabilizer_usb_2 3.38 mm to (191.5, 44.0)
- moved J16 2.06 mm to (149.6, 62.2)
Connections:
- J16 pad 6: unconnected-(J16-Pin_6-Pad6) -> /Solar_Pos_In
Routing:
- net /Solar_Pos_In: track 0.00 -> 20.7 mm
- net /SDA: track 95.7 -> 89.9 mm
- net /BATpos: track 82.8 -> 86.2 mm
- net /Solarpos: track 40.2 -> 37.5 mm
- net /SCL: track 87.2 -> 89.4 mm, vias 0 -> 1
- net /3.3V: track 110.5 -> 108.8 mm
Other:
- board text added: "Solar Panel +"
- board text added: "Solar Panel -"
- board text added: "Solar_In"
- board text added: "Solar_Out"
- board text removed: "GND_Solar"

Commit message: updated pcb design
Parts:
- added Bat_Connector1: Battery, TerminalBlock:TerminalBlock_Xinya_XY308-2.54-2P_1x02_P2.54mm_Horizontal, F.Cu at (198.6, 74.0)
- moved m3-br 48.0 mm to (197.1, 46.5)
- moved m3-tr 35.4 mm to (197.1, 91.5)
- moved m3-tl 35.4 mm to (117.1, 46.5)
- moved m3-bl 7.70 mm to (117.1, 91.5)
- moved J20 0.65 mm to (150.9, 94.5)
Routing:
- net /3.3V: track 108.8 -> 86.9 mm, vias 0 -> 2
- net /BATpos: track 86.2 -> 101.6 mm
- net /BATneg: vias 52 -> 51
Other:
- board size 76 x 56 mm -> 90 x 55 mm
