File: pcb-design/scale module/_V0_3-Scale_Module.kicad_sch (KiCad schematic)
At the start: 24 parts, among them J1 ESP32-left-RXTX, J10 PowerIn, J11 Loadcell1-Input, J12 Loadcell2-Input, J13 DS18B20-1, J14 DS18B20-2, J15 SHT40 Ambient, J16 Sound Module INMP441 - Hive2, J17 I2C, J18 Expansion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

Commit message: updated pcb design
Parts:
- removed J14: DS18B20-2, TerminalBlock:TerminalBlock_Xinya_XY308-2.54-3P_1x03_P2.54mm_Horizontal, symbol Connector_Generic:Conn_01x03
- added H1, H2, H3, H4: MountingHole, MountingHole:MountingHole_3.2mm_M3, symbol Mechanical:MountingHole
- J11, J12: footprint TerminalBlock:TerminalBlock_Xinya_XY308-2.54-12P_1x12_P2.54mm_Horizontal -> Connector_JST:JST_XH_B5B-XH-A_1x05_P2.50mm_Vertical; symbol Connector_Generic:Conn_01x12 -> Connector_Generic:Conn_01x05
- J13: footprint TerminalBlock:TerminalBlock_Xinya_XY308-2.54-3P_1x03_P2.54mm_Horizontal -> Connector_JST:JST_XH_B3B-XH-A_1x03_P2.50mm_Vertical
- J15, J20: footprint TerminalBlock:TerminalBlock_Xinya_XY308-2.54-4P_1x04_P2.54mm_Horizontal -> Connector_JST:JST_XH_B4B-XH-A_1x04_P2.50mm_Vertical
- J16, J6: footprint TerminalBlock:TerminalBlock_Xinya_XY308-2.54-6P_1x06_P2.54mm_Horizontal -> Connector_JST:JST_XH_B6B-XH-A_1x06_P2.50mm_Vertical
Connections:
- net 3.3V: now also J9.1 (Pin_1); no longer J9.2 (Pin_2)
- net GND: now also J11.1 (Pin_1), J12.1 (Pin_1), J9.6 (Pin_6); no longer J9.1 (Pin_1)
- net GPIO18: now also J9.4 (Pin_4); no longer J9.5 (Pin_5)
- net GPIO19: now also J9.3 (Pin_3); no longer J9.4 (Pin_4)
- net GPIO23: now also J9.5 (Pin_5); no longer J9.3 (Pin_3)
- net GPIO5: now also J9.2 (Pin_2); no longer J9.6 (Pin_6)
- net at J12.2 (Pin_2): now also J8.1 (Pin_1); no longer J12.1 (Pin_1)
- net at J8.2 (Pin_2): now also J12.3 (Pin_3); no longer J12.10 (Pin_10)
- net at J8.3 (Pin_3): now also J12.4 (Pin_4); no longer J12.11 (Pin_11)
- net at J8.4 (Pin_4): now also J12.5 (Pin_5); no longer J12.12 (Pin_12)
- net at J7.1 (Pin_1): now also J11.2 (Pin_2); no longer J11.9 (Pin_9)
- net at J7.2 (Pin_2): now also J11.3 (Pin_3); no longer J11.10 (Pin_10)
- net at J7.3 (Pin_3): now also J11.4 (Pin_4); no longer J11.11 (Pin_11)
- net at J7.4 (Pin_4): now also J11.5 (Pin_5); no longer J11.12 (Pin_12)
Other:
- note removed: "DS18B20 Hive2"
