File: pcb-design/esp32-c6 (recommended design)/_V0_5-Scale_Module.kicad_pcb (KiCad board)
At the start: 2 copper layers, 60 x 90 mm, 32 parts, among them J1 Conn_01x01_Socket, J10 PowerIn, J11 PowerIn, J12 BatIN, J13 DS18B20, J15 SHT40 Ambient, J18 TPS63020-GND-OUT, J19 PowerModuleHeader, J2 Conn_01x01_Socket, J20 TPS63020-V-IN, J21 NAU7802, J22 MAXS17048, J23 TPS63020-3.3V-OUT, J3 PowerSelector, J5 RTC, J6 TPS63020-GND-IN, J9 SD-Module, SW1 SW_Push, U1 113991254

Commit message: added pins for 2nd pushbutton to PCB
Parts:
- added SET: Setup_Button, Connector_PinSocket_2.54mm:PinSocket_1x02_P2.54mm_Vertical, F.Cu at (187.5, 106.5)
- INSP: renamed from SW1; value SW_Push -> Inspection_Button
Routing:
- net /D0: track 0.00 -> 6.03 mm
- net GND: vias 68 -> 69
Other:
- board text removed: "D4"
- board text removed: "D5"
