File: pcb-design/esp32-c6 (recommended design)/_V0_5-Scale_Module.kicad_sch (KiCad schematic)
At the start: 32 parts, among them J1 Conn_01x01_Socket, J10 PowerIn, J11 PowerIn, J12 BatIN, J13 DS18B20, J15 SHT40 Ambient, J18 TPS63020-GND-OUT, J19 PowerModuleHeader, J2 Conn_01x01_Socket, J20 TPS63020-V-IN, J21 NAU7802, J22 MAXS17048, J23 TPS63020-3.3V-OUT, J3 PowerSelector, J5 RTC, J6 TPS63020-GND-IN, J9 SD-Module, SW1 SW_Push, U1 113991254

Commit message: added pins for 2nd pushbutton to PCB
Parts:
- added SW2: Setup_Button, Connector_PinSocket_2.54mm:PinSocket_1x02_P2.54mm_Vertical, symbol Switch:SW_Push
- SW1: value SW_Push -> Inspection_Button
Connections:
- net D0: now also SW2.2
- net GND: now also SW2.1
Changed lines of the file:
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@@
 		)
 	)
+	(label "GND"
+		(at 133.35 167.64 180)
+		(effects
+			(font
+				(size 1.27 1.27)
+			)
+			(justify right bottom)
+		)
+	)
 	(label "D0"
 		(at 40.64 133.35 180)
@@
 		)
 	)
+	(label "D0"
+		(at 143.51 167.64 0)
+		(effects
+			(font
+				(size 1.27 1.27)
+			)
+			(justify left bottom)
+		)
+	)
 	(label "GND"
 		(at 22.86 180.34 180)
@@
 		)
 		(instances
-			(project "_V0_4-Scale_Module"
+			(project "_V0_5-Scale_Module"
 				(path "/0fd72f3f-0d89-4c92-9f9e-d7a48828e0f6"
 					(reference "J12")
@@
 	)
 	(symbol
+		(lib_id "Switch:SW_Push")
+		(at 138.43 167.64 0)
+		(unit 1)
+		(body_style 1)
+		(exclude_from_sim no)
+		(in_bom yes)
+		(on_board yes)
+		(in_pos_files yes)
+		(dnp no)
+		(fields_autoplaced yes)
+		(property "Reference" "SW2"
+			(at 138.43 160.02 0)
+			(show_name no)
+			(do_not_autoplace no)
+			(effects
+				(font
+					(size 1.27 1.27)
+				)
+			)
+		)
+		(property "Value" "Setup_Button"
+			(at 138.43 162.56 0)
+			(show_name no)
+			(do_not_autoplace no)
+			(effects
+				(font
+					(face "Standard Symbols PS")
+					(size 1.27 1.27)
+				)
+			)
+		)
+		(property "Footprint" "Connector_PinSocket_2.54mm:PinSocket_1x02_P2.54mm_Vertical"
+			(at 138.43 162.56 0)
+			(hide yes)
+			(show_name no)
+			(do_not_autoplace no)
+			(effects
+				(font
+					(size 1.27 1.27)
+				)
+			)
+		)
+		(property "Datasheet" ""
+			(at 138.43 162.56 0)
+			(hide yes)
+			(show_name no)
+			(do_not_autoplace no)
+			(effects
+				(font
+					(size 1.27 1.27)
+				)
+			)
+		)
+		(property "Description" "Push button switch, generic, two pins"
+			(at 138.43 167.64 0)
+			(hide yes)
+			(show_name no)
+			(do_not_autoplace no)
+			(effects
+				(font
+					(size 1.27 1.27)
+				)
+			)
+		)
+		(pin "1"
+		)
+		(pin "2"
+		)
+		(instances
+			(project "_V0_5-Scale_Module"
+				(path "/0fd72f3f-0d89-4c92-9f9e-d7a48828e0f6"
+					(reference "SW2")
+					(unit 1)
+				)
+			)
+		)
+	)
+	(symbol
 		(lib_id "Mechanical:MountingHole")
 		(at 73.66 87.63 0)
@@
 		)
 		(instances
-			(project "_V0_4-Scale_Module"
+			(project "_V0_5-Scale_Module"
 				(path "/0fd72f3f-0d89-4c92-9f9e-d7a48828e0f6"
 					(reference "H8")
@@
 		)
 		(instances
-			(project "_V0_4-Scale_Module"
+			(project "_V0_5-Scale_Module"
 				(path "/0fd72f3f-0d89-4c92-9f9e-d7a48828e0f6"
 					(reference "J21")
@@
 		)
 		(instances
-			(project "_V0_4-Scale_Module"
+			(project "_V0_5-Scale_Module"
 				(path "/0fd72f3f-0d89-4c92-9f9e-d7a48828e0f6"
 					(reference "J10")
@@
 		)
 		(instances
-			(project "_V0_4-Scale_Module"
+			(project "_V0_5-Scale_Module"
 				(path "/0fd72f3f-0d89-4c92-9f9e-d7a48828e0f6"
 					(reference "J18")
@@
 		)
 		(instances
-			(project "_V0_4-Scale_Module"
+			(project "_V0_5-Scale_Module"
 				(path "/0fd72f3f-0d89-4c92-9f9e-d7a48828e0f6"
 					(reference "J19")
@@
 		)
 		(instances
-			(project "_V0_4-Scale_Module"
+			(project "_V0_5-Scale_Module"
 				(path "/0fd72f3f-0d89-4c92-9f9e-d7a48828e0f6"
 					(reference "#FLG01")
@@
 		)
 		(instances
-			(project "_V0_4-Scale_Module"
+			(project "_V0_5-Scale_Module"
 				(path "/0fd72f3f-0d89-4c92-9f9e-d7a48828e0f6"
 					(reference "i2c1")
@@
 		)
 		(instances
-			(project "_V0_4-Scale_Module"
+			(project "_V0_5-Scale_Module"
 				(path "/0fd72f3f-0d89-4c92-9f9e-d7a48828e0f6"
 					(reference "J9")
@@
 		)
 		(instances
-			(project "_V0_4-Scale_Module"
+			(project "_V0_5-Scale_Module"
 				(path "/0fd72f3f-0d89-4c92-9f9e-d7a48828e0f6"
 					(reference "J5")
@@
 		)
 		(instances
-			(project "_V0_4-Scale_Module"
+			(project "_V0_5-Scale_Module"
 				(path "/0fd72f3f-0d89-4c92-9f9e-d7a48828e0f6"
 					(reference "H4")
@@
 		)
 		(instances
-			(project "_V0_4-Scale_Module"
+			(project "_V0_5-Scale_Module"
 				(path "/0fd72f3f-0d89-4c92-9f9e-d7a48828e0f6"
 					(reference "MAX17048")
@@
 		)
 		(instances
-			(project "_V0_4-Scale_Module"
+			(project "_V0_5-Scale_Module"
 				(path "/0fd72f3f-0d89-4c92-9f9e-d7a48828e0f6"
 					(reference "J20")
@@
 		)
 		(instances
-			(project "_V0_4-Scale_Module"
+			(project "_V0_5-Scale_Module"
 				(path "/0fd72f3f-0d89-4c92-9f9e-d7a48828e0f6"
 					(reference "SCL-4.7k1")
@@
 		)
 		(instances
-			(project "_V0_4-Scale_Module"
+			(project "_V0_5-Scale_Module"
 				(path "/0fd72f3f-0d89-4c92-9f9e-d7a48828e0f6"
 					(reference "TP4056+1")
@@
 		)
 		(instances
-			(project "_V0_4-Scale_Module"
+			(project "_V0_5-Scale_Module"
 				(path "/0fd72f3f-0d89-4c92-9f9e-d7a48828e0f6"
 					(reference "1W-4.7k1")
@@
 		)
 		(instances
-			(project "_V0_4-Scale_Module"
+			(project "_V0_5-Scale_Module"
 				(path "/0fd72f3f-0d89-4c92-9f9e-d7a48828e0f6"
 					(reference "J3")
@@
 		)
 		(instances
-			(project "_V0_4-Scale_Module"
+			(project "_V0_5-Scale_Module"
 				(path "/0fd72f3f-0d89-4c92-9f9e-d7a48828e0f6"
 					(reference "J23")
@@
 		)
 		(instances
-			(project "_V0_4-Scale_Module"
+			(project "_V0_5-Scale_Module"
 				(path "/0fd72f3f-0d89-4c92-9f9e-d7a48828e0f6"
 					(reference "J13")
@@
 			)
 		)
-		(property "Value" "SW_Push"
+		(property "Value" "Inspection_Button"
 			(at 119.38 162.56 0)
 			(show_name no)
@@
 		)
 		(instances
-			(project "_V0_4-Scale_Module"
+			(project "_V0_5-Scale_Module"
 				(path "/0fd72f3f-0d89-4c92-9f9e-d7a48828e0f6"
 					(reference "SW1")
@@
 		)
 		(instances
-			(project "_V0_4-Scale_Module"
+			(project "_V0_5-Scale_Module"
 				(path "/0fd72f3f-0d89-4c92-9f9e-d7a48828e0f6"
 					(reference "J11")
@@
 		)
 		(instances
-			(project "_V0_4-Scale_Module"
+			(project "_V0_5-Scale_Module"
 				(path "/0fd72f3f-0d89-4c92-9f9e-d7a48828e0f6"
 					(reference "J2")
@@
 		)
 		(instances
-			(project "_V0_4-Scale_Module"
+			(project "_V0_5-Scale_Module"
 				(path "/0fd72f3f-0d89-4c92-9f9e-d7a48828e0f6"
 					(reference "SDA-4.7k1")
@@
 		)
 		(instances
-			(project "_V0_4-Scale_Module"
+			(project "_V0_5-Scale_Module"
 				(path "/0fd72f3f-0d89-4c92-9f9e-d7a48828e0f6"
 					(reference "H3")
@@
 		)
 		(instances
-			(project "_V0_4-Scale_Module"
+			(project "_V0_5-Scale_Module"
 				(path "/0fd72f3f-0d89-4c92-9f9e-d7a48828e0f6"
 					(reference "U1")
@@
 		)
 		(instances
-			(project "_V0_4-Scale_Module"
+			(project "_V0_5-Scale_Module"
 				(path "/0fd72f3f-0d89-4c92-9f9e-d7a48828e0f6"
 					(reference "#PWR01")
@@
 		)
 		(instances
-			(project "_V0_4-Scale_Module"
+			(project "_V0_5-Scale_Module"
 				(path "/0fd72f3f-0d89-4c92-9f9e-d7a48828e0f6"
 					(reference "J6")
@@
 		)
 		(instances
-			(project "_V0_4-Scale_Module"
+			(project "_V0_5-Scale_Module"
 				(path "/0fd72f3f-0d89-4c92-9f9e-d7a48828e0f6"
 					(reference "H1")
@@
 		)
 		(instances
-			(project "_V0_4-Scale_Module"
+			(project "_V0_5-Scale_Module"
 				(path "/0fd72f3f-0d89-4c92-9f9e-d7a48828e0f6"
 					(reference "H2")
@@
 		)
 		(instances
-			(project "_V0_4-Scale_Module"
+			(project "_V0_5-Scale_Module"
 				(path "/0fd72f3f-0d89-4c92-9f9e-d7a48828e0f6"
 					(reference "TP4056-1")
@@
 		)
 		(instances
-			(project "_V0_4-Scale_Module"
+			(project "_V0_5-Scale_Module"
 				(path "/0fd72f3f-0d89-4c92-9f9e-d7a48828e0f6"
 					(reference "J1")
@@
 		)
 		(instances
-			(project "_V0_4-Scale_Module"
+			(project "_V0_5-Scale_Module"
 				(path "/0fd72f3f-0d89-4c92-9f9e-d7a48828e0f6"
 					(reference "J22")
@@
 		)
 		(instances
-			(project "_V0_4-Scale_Module"
+			(project "_V0_5-Scale_Module"
 				(path "/0fd72f3f-0d89-4c92-9f9e-d7a48828e0f6"
 					(reference "J15")
@@
 		)
 		(instances
-			(project "_V0_4-Scale_Module"
+			(project "_V0_5-Scale_Module"
 				(path "/0fd72f3f-0d89-4c92-9f9e-d7a48828e0f6"
 					(reference "H6")
